File: hardware/logicboard/p2m-001.brd (EAGLE design)
At the start: 72 x 72 mm, 68 parts, among them IC1 74LS06N, IC101 74LS153D, IC102 LTC485S, IC103 LTC485S, IC2 4066N, J1 MKR, J101 Qwiic, J102 Qwiic, J103 Qwiic, J104 Qwiic, J2 GPIO, J4 3-PIN SMD, J5 SPI, J6 LED, K1 G5V1, T1 2SC1815, U1 DS18B20

Commit message: First try.
Parts:
- removed C101, C102, C103: 10n, rcl:C2012
- removed C8: 10n, resistor:C025-024X044
- removed C9: 100n, rcl:C025-024X044
- removed D2: (no value), SparkFun-DiscreteSemi:DIODE-1N4148
- removed H1, H2: STAND-OFF, SparkFun-Hardware:STAND-OFF
- removed IC101: 74LS153D, 74xx-us:SO16
- removed IC102, IC103: LTC485S, linear-technology:SOIC8
- removed IN, RX, V+, VIN, VO, VOR: (no value), wirepad:SMD1,27-2,54
- removed J101, J102, J103, J104: Qwiic, SparkFun-Connectors:1X04_1MM_RA
- removed J2: GPIO, SparkFun-Connectors:JST-4-PTH
- removed J20: (no value), SparkFun-Connectors:1X04_1.27MM
- removed J5: SPI, SparkFun-Connectors:1X06_1.27MM
- removed J6: LED, SparkFun-Connectors:JST-3-PTH
- removed JP0: GNDPIN, pinhead:1X01
- removed JP2: RTC, SparkFun-Connectors:1X05
- removed JP3: MPXJMP, pinhead:1X02
- removed JP5: PWR, pinhead:1X03
- removed JP6: LED, pinhead:1X03
- removed K1: G5V1, relay:G5V1
- removed R1: 1k, resistor:0204/5
- removed R101: 10k, rcl:M2012
- removed R102, R103: 120, rcl:M2012
- removed R2: 47k, resistor:0204/5
- removed SV1: (no value), con-ml:ML16L
- removed SV2: (no value), con-ml:ML20L
- removed T1: 2SC1815, transistor:TO92-ECB
- added J3: (no value), SparkFun-Connectors:1X10-2MM
- J4: value 3-PIN SMD -> (none); device SparkFun-Connectors:JST-3-SMD -> SparkFun-Connectors:JST-4-PTH
- moved J4 69.5 mm to (23.5, 66.0), flipped to the top, turned to 0 degrees
- moved C10 57.6 mm to (4.00, 24.0), turned to 0 degrees
- moved R3 55.3 mm to (10.0, 24.0), turned to 180 degrees
- moved C4 54.0 mm to (5.00, 20.0)
- moved U1 52.5 mm to (9.50, 3.50)
- moved JP1 47.8 mm to (32.0, 12.0)
- moved V1 42.0 mm to (15.8, 12.0), turned to 90 degrees
- moved C5 41.5 mm to (10.0, 46.0)
- moved C3 39.8 mm to (11.0, 20.0)
- moved R4 38.4 mm to (17.0, 24.0)
- moved C7 35.8 mm to (21.0, 59.0), turned to 0 degrees
- moved D3 35.1 mm to (21.0, 62.0), turned to 0 degrees
- moved C6 32.4 mm to (21.0, 45.0)
- moved J1 31.8 mm to (35.0, 66.0), turned to 0 degrees
- moved IC1 31.3 mm to (21.0, 34.0)
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Connections:
- removed net MRX: IC101.6, IC102.1
- removed net MRX+: IC102.6, R102.1, SV2.6
- removed net MRX-: IC102.7, R102.2, SV2.8
- removed net MTX+: IC103.6, R103.1, SV2.10
- removed net MTX-: IC103.7, R103.2, SV2.12
- removed net NDX: IC101.14, R101.1, SV2.4
- removed net RLYDRV: R1.1, R2.2, T1.B
- removed net RLYOUT: J4.1, K1.10
- removed net RLYSNK: D2.A, K1.9, T1.C
- removed net VOUTRAW2: F1.1, J4.3, K1.1, VO.1
- net ANLG0R: no longer SV1.3
- net ANLG1R: no longer SV1.7
- net ANLG2R: no longer SV1.11
- net ANLG3R: no longer SV1.15
- net DTCT0: no longer SV1.2
- net DTCT1: no longer SV1.6
- net DTCT2: no longer SV1.10
- net DTCT3: no longer SV1.14
- net GND: no longer C101.2, C102.2, C103.2, C8.2, C9.2, IC101.1, IC101.10, IC101.11, IC101.12, IC101.13, IC101.15, IC101.2, IC101.3, IC101.4, IC101.8, IC102.2, IC102.3, IC102.4, IC102.5, IC103.5, J101.1, J102.1, J103.1, J104.1, J2.1, J5.6, J6.2, JP0.1, JP2.2, JP5.1, JP6.2, R2.1, SV1.1, SV1.13, SV1.5, SV1.9, SV2.1, SV2.15, SV2.16, SV2.5, T1.E
- net GPIO0: no longer J2.3, J20.3
- net GPIO1: no longer J2.4, J20.4
- net LED0: no longer SV2.7
- net LED0A: no longer J6.1, JP6.1
- net LED1: no longer SV2.20
- net LED1A: no longer J6.3, JP6.3
- net MIN: no longer IC101.5, IN.1, JP3.2, OK1.7
- net MIRTN: no longer SV2.11
- net MISND: no longer SV2.9
- net MISO: no longer J5.1
- net MORTN: no longer SV2.17
- net MOSI: no longer J5.4
- net MOSND: no longer SV2.13
- net MTRTN: no longer SV2.18
- net MTSND: no longer SV2.14
- net RLY: no longer R1.2
- net RST: no longer J5.5, SV2.3
- net RX: now also OK1.7; no longer IC101.7, JP3.1, RX.1
- net SCK: no longer J5.3
- net SCL: no longer J101.4, J102.4, J103.4, J104.4, JP2.4
- net SDA: no longer J101.3, J102.3, J103.3, J104.3, JP2.5
- net TX: no longer IC103.4
- net V+: no longer JP5.3, SV2.2, V+.1
- net VCC: no longer C101.1, C102.1, C103.1, C8.1, C9.1, D2.C, IC101.16, IC102.8, IC103.2, IC103.3, IC103.8, J101.2, J102.2, J103.2, J104.2, J2.2, J5.2, JP2.1, JP5.2, K1.2, R101.2, SV2.19
- net VCC/2: no longer SV1.12, SV1.16, SV1.4, SV1.8
- net VIN: no longer VIN.1
- net VOUTRAW: now also F1.1; no longer J4.2, K1.5, K1.6, VOR.1
Routing:
- net GND: track 423.9 -> 169.0 mm, vias 4 -> 1
- net VCC: track 400.8 -> 160.5 mm, vias 18 -> 3
- net SDA: track 214.5 -> 79.4 mm, vias 5 -> 1
- net MRX+: track 119.0 -> 0.00 mm, vias 4 -> 0
- net MISO: track 117.0 -> 0.00 mm, vias 1 -> 0
- net V+: track 149.6 -> 33.9 mm, vias 2 -> 0
- net MIN: track 114.1 -> 0.00 mm, vias 6 -> 0
- net SCK: track 111.7 -> 0.00 mm, vias 3 -> 0
- net LED0A: track 110.6 -> 0.00 mm, vias 2 -> 0
- net MOSI: track 107.5 -> 0.00 mm, vias 1 -> 0
- net SCL: track 180.4 -> 80.7 mm, vias 9 -> 0
- net RST: track 112.5 -> 15.3 mm, vias 9 -> 0
- net MORTN: track 91.2 -> 0.00 mm, vias 3 -> 0
- net VOUT: track 100.4 -> 11.2 mm, vias 2 -> 0
- net GPIO0: track 82.2 -> 0.00 mm, vias 4 -> 0
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- removed copper zone on layer 1, net GND
- removed copper zone on layer 16, net GND
Other:
- board size 72 x 72 mm -> 47 x 72 mm
- board text added: "0.0.1-X"
- board text added: "Pineapple IIm"
- board text removed: "(3V3)"
- board text removed: "(JP4)"
- board text removed: "(OUT2)"
- board text removed: "+"
- board text removed: "2.7.1-GM"
- board text removed: "5V"
- board text removed: "Close Here"
- board text removed: "GeekPort II"
- board text removed: "Min. requirement for MIDI IN"
- board text removed: "Min. requirement for MIDI OUT"
- board text removed: "PWR"
- board text removed: "Pineapple II"
- board text removed: "RTC1"
- board text removed: "SPI"
- board text removed: "SparkFun Real Time Clock Module (12708)"
- board text removed: "This pin pulls up U1"

Commit message: Second try.
Parts:
- removed R5: 102, resistor:0204/5
- added J2: (no value), SparkFun-Connectors:JST-4-PTH
- moved U$1 42.0 mm to (10.0, 0.50), flipped to the top
- moved LOGO1 33.1 mm to (39.0, 3.00)
- moved U1 16.3 mm to (6.50, 19.5)
- moved D1 10.0 mm to (32.0, 6.50)
- moved C4 9.00 mm to (14.0, 20.0), turned to 270 degrees
- moved C3 6.00 mm to (17.0, 20.0), turned to 90 degrees
- moved R4 4.12 mm to (21.0, 25.0)
- moved C2 2.00 mm to (20.0, 20.0), turned to 90 degrees
- moved C5 1.00 mm to (10.0, 45.0)
- moved C6 1.00 mm to (21.0, 46.0)
- moved C7 1.00 mm to (21.0, 60.0)
- moved D3 1.00 mm to (21.0, 63.0)
- moved F1 1.00 mm to (24.0, 11.0)
- moved IC1 1.00 mm to (21.0, 35.0)
- moved IC2 1.00 mm to (10.0, 34.0)
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Connections:
- removed net LED1A: R5.1
- new net LDE0A: J3.5
- net ANLG0: now also J4.3
- net DTCT0: now also J4.4
- net GND: now also J2.1, J3.1, J3.4, J3.9, J4.1
- net GPIO0: now also J2.3
- net GPIO1: now also J2.4
- net LED1: no longer R5.2
- net MIRTN: now also J3.7
- net MISND: now also J3.6
- net MORTN: now also J3.10
- net MOSND: now also J3.8
- net RST: now also J3.3
- net V+: now also J3.2
- net VCC: now also J2.2
- net VCC/2: now also J4.2
Routing:
- net MISND: track 0.00 -> 103.8 mm, vias 0 -> 1
- net MIRTN: track 9.50 -> 93.7 mm, vias 0 -> 1
- net MOSND: track 0.00 -> 76.7 mm, vias 0 -> 4
- net MORTN: track 0.00 -> 69.3 mm, vias 0 -> 3
- net GND: track 169.0 -> 223.0 mm, vias 1 -> 2
- net ANLG0: track 48.7 -> 101.1 mm
- net LED1: track 49.9 -> 0.00 mm
- net GPIO1: track 0.00 -> 44.6 mm
- net GPIO0: track 0.00 -> 34.7 mm
- net RST: track 15.3 -> 48.9 mm
- net THS: track 112.9 -> 83.4 mm, vias 1 -> 0
- net DTCT0: track 0.00 -> 28.0 mm
- net D7GATE: track 70.2 -> 95.6 mm, vias 3 -> 2
- net VCC: track 160.5 -> 185.2 mm, vias 3 -> 4
- net RX: track 57.6 -> 71.5 mm, vias 0 -> 1
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