File: hardware/logicboard/p2m-001.sch (EAGLE design)
At the start: 68 parts, among them IC1 74LS06N, IC101 74LS153D, IC102 LTC485S, IC103 LTC485S, IC2 4066N, J1 MKR, J101 Qwiic, J102 Qwiic, J103 Qwiic, J104 Qwiic, J2 GPIO, J4 3-PIN SMD, J5 SPI, J6 LED, K1 G5V1, T1 2SC1815, U1 DS18B20

Commit message: First try.
Parts:
- removed C101, C102, C103: 10n, rcl:C-EUC2012
- removed C8: 10n, resistor:C-EU025-024X044
- removed C9: 100n, rcl:C-EU025-024X044
- removed D2: DIODE-1N4148, SparkFun-DiscreteSemi:DIODE-1N4148
- removed H1, H2: STAND-OFF, SparkFun-Hardware:STAND-OFF
- removed IC101: 74LS153D, 74xx-us:74LS153D
- removed IC102, IC103: LTC485S, linear-technology:LTC485S
- removed IN, RX, V+, VIN, VO, VOR: (no value), wirepad:SMD2
- removed J101, J102, J103, J104: Qwiic, SparkFun-Connectors:QWIIC_CONNECTORJS-1MM
- removed J2: GPIO, SparkFun-Connectors:CONN_04JST-PTH
- removed J20: (no value), SparkFun-Connectors:CONN_041.27MM
- removed J5: SPI, SparkFun-Connectors:CONN_061.27MM
- removed J6: LED, SparkFun-Connectors:CONN_03JST-PTH
- removed JP0: GNDPIN, pinhead:PINHD-1X1
- removed JP2: RTC, SparkFun-Connectors:CONN_05
- removed JP3: MPXJMP, pinhead:PINHD-1X2
- removed JP5: PWR, pinhead:PINHD-1X3
- removed JP6: LED, pinhead:PINHD-1X3
- removed K1: G5V1, relay:G5V1
- removed R1: 1k, resistor:R-EU_0204/5
- removed R101: 10k, rcl:R-EU_M2012
- removed R102, R103: 120, rcl:R-EU_M2012
- removed R2: 47k, resistor:R-EU_0204/5
- removed SV1: (no value), con-ml:ML16LE
- removed SV2: (no value), con-ml:ML20LE
- removed T1: 2SC1815, transistor:2SC1815
- added J3: (no value), SparkFun-Connectors:CONN_102MM
- J4: value 3-PIN SMD -> (none); device SparkFun-Connectors:CONN_03JST-SMD -> SparkFun-Connectors:CONN_04JST-PTH
Connections:
- removed net MRX: IC101A.1C0, IC102.RO
- removed net MRX+: IC102.A, R102.1, SV2-6.S
- removed net MRX-: IC102.B, R102.2, SV2-8.S
- removed net MTX+: IC103.A, R103.1, SV2-10.S
- removed net MTX-: IC103.B, R103.2, SV2-12.S
- removed net NDX: IC101A.A, R101.1, SV2-4.S
- removed net RLYDRV: R1.1, R2.2, T1.B
- removed net RLYOUT: J4.1, K12.S
- removed net RLYSNK: D2.A, K11.2, T1.C
- removed net VOUTRAW2: F1.1, J4.3, K12.O, VO.P
- net ANLG0R: no longer SV1-3.S
- net ANLG1R: no longer SV1-7.S
- net ANLG2R: no longer SV1-11.S
- net ANLG3R: no longer SV1-15.S
- net DTCT0: no longer SV1-2.S
- net DTCT1: no longer SV1-6.S
- net DTCT2: no longer SV1-10.S
- net DTCT3: no longer SV1-14.S
- net GND: no longer C101.2, C102.2, C103.2, C8.2, C9.2, IC101A.1C2, IC101A.1C3, IC101A.1G, IC101A.2C0, IC101A.2C1, IC101A.2C2, IC101A.2C3, IC101A.2G, IC101A.B, IC102.!RE, IC102.DE, IC102.DI, IC102.GND, IC103.GND, J101.GND, J102.GND, J103.GND, J104.GND, J2.1, J5.6, J6.2, JP0.1, JP2.2, JP5.1, JP6.2, R2.1, SV1-1.S, SV1-13.S, SV1-5.S, SV1-9.S, SV2-1.S, SV2-15.S, SV2-16.S, SV2-5.S, T1.E
- net GPIO0: no longer J2.3, J20.3
- net GPIO1: no longer J2.4, J20.4
- net LED0: no longer SV2-7.S
- net LED0A: no longer J6.1, JP6.1
- net LED1: no longer SV2-20.S
- net LED1A: no longer J6.3, JP6.3
- net MIN: no longer IC101A.1C1, IN.P, JP3.2, OK1A.VO1
- net MIRTN: no longer SV2-11.S
- net MISND: no longer SV2-9.S
- net MISO: no longer J5.1
- net MORTN: no longer SV2-17.S
- net MOSI: no longer J5.4
- net MOSND: no longer SV2-13.S
- net MTRTN: no longer SV2-18.S
- net MTSND: no longer SV2-14.S
- net RLY: no longer R1.2
- net RST: no longer J5.5, SV2-3.S
- net RX: now also OK1A.VO1; no longer IC101A.1Y, JP3.1, RX.P
- net SCK: no longer J5.3
- net SCL: no longer J101.SCL, J102.SCL, J103.SCL, J104.SCL, JP2.4
- net SDA: no longer J101.SDA, J102.SDA, J103.SDA, J104.SDA, JP2.5
- net TX: no longer IC103.DI
- net V+: no longer JP5.3, SV2-2.S, V+.P
- net VCC: no longer C101.1, C102.1, C103.1, C8.1, C9.1, D2.C, IC102.VCC, IC103.!RE, IC103.DE, IC103.VCC, J101.VCC, J102.VCC, J103.VCC, J104.VCC, J2.2, J5.2, JP2.1, JP5.2, K11.1, R101.2, SV2-19.S
- net VCC/2: no longer SV1-12.S, SV1-16.S, SV1-4.S, SV1-8.S
- net VIN: no longer VIN.P
- net VOUTRAW: now also F1.1; no longer J4.2, K12.P, K12.P@1, VOR.P
Other:
- note removed: "BackPort 2.0"

Commit message: Second try.
Parts:
- removed R5: 102, resistor:R-EU_0204/5
- added J2: (no value), SparkFun-Connectors:CONN_04JST-PTH
Connections:
- removed net LED1A: R5.1
- new net LDE0A: J3.5
- net ANLG0: now also J4.3
- net DTCT0: now also J4.4
- net GND: now also J2.1, J3.1, J3.4, J3.9, J4.1
- net GPIO0: now also J2.3
- net GPIO1: now also J2.4
- net LED1: no longer R5.2
- net MIRTN: now also J3.7
- net MISND: now also J3.6
- net MORTN: now also J3.10
- net MOSND: now also J3.8
- net RST: now also J3.3
- net V+: now also J3.2
- net VCC: now also J2.2
- net VCC/2: now also J4.2
Other:
- moved on the sheet: J3
Changed lines of the file:
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@@
 <part name="SUPPLY29" library="supply2" deviceset="GND" device=""/>
 <part name="J1" library="SparkFun-Connectors" library_urn="urn:adsk.eagle:library:513" deviceset="CONN_05" device="JST" package3d_urn="urn:adsk.eagle:package:38120/1" value="MKR"/>
-<part name="R5" library="resistor" library_urn="urn:adsk.eagle:library:348" deviceset="R-EU_" device="0204/5" package3d_urn="urn:adsk.eagle:package:23488/1" value="102"/>
 <part name="SUPPLY33" library="supply2" deviceset="GND" device=""/>
 <part name="XMC1_SS" library="wirepad" library_urn="urn:adsk.eagle:library:412" deviceset="PAD-N" device=""/>
@@
 <part name="J3" library="SparkFun-Connectors" library_urn="urn:adsk.eagle:library:513" deviceset="CONN_10" device="2MM" package3d_urn="urn:adsk.eagle:package:38158/1"/>
 <part name="J4" library="SparkFun-Connectors" library_urn="urn:adsk.eagle:library:513" deviceset="CONN_04" device="JST-PTH" package3d_urn="urn:adsk.eagle:package:38101/1"/>
+<part name="J2" library="SparkFun-Connectors" library_urn="urn:adsk.eagle:library:513" deviceset="CONN_04" device="JST-PTH" package3d_urn="urn:adsk.eagle:package:38101/1"/>
 </parts>
 <sheets>
@@
 <attribute name="NAME" x="58.42" y="55.88" size="1.778" layer="95" rot="R90" align="bottom-center"/>
 </instance>
-<instance part="R5" gate="G$1" x="274.32" y="109.22" smashed="yes">
-<attribute name="NAME" x="274.32" y="111.76" size="1.778" layer="95" align="bottom-center"/>
-<attribute name="VALUE" x="279.4" y="111.76" size="1.778" layer="96" align="bottom-center"/>
-</instance>
 <instance part="SUPPLY33" gate="GND" x="35.56" y="220.98" smashed="yes"/>
 <instance part="XMC1_SS" gate="G$1" x="96.52" y="195.58" smashed="yes"/>
@@
 <instance part="SUPPLY1" gate="GND" x="236.22" y="35.56" smashed="yes"/>
 <instance part="SUPPLY6" gate="GND" x="259.08" y="83.82" smashed="yes"/>
-<instance part="J3" gate="G$1" x="312.42" y="142.24" smashed="yes">
-<attribute name="VALUE" x="312.42" y="119.634" size="1.778" layer="96" font="vector"/>
-<attribute name="NAME" x="312.42" y="150.368" size="1.778" layer="95" font="vector"/>
+<instance part="J3" gate="G$1" x="309.88" y="142.24" smashed="yes">
+<attribute name="VALUE" x="309.88" y="119.634" size="1.778" layer="96" font="vector"/>
+<attribute name="NAME" x="309.88" y="150.368" size="1.778" layer="95" font="vector"/>
 </instance>
 <instance part="J4" gate="G$1" x="314.96" y="101.6" smashed="yes">
 <attribute name="VALUE" x="309.88" y="94.234" size="1.778" layer="96" font="vector"/>
 <attribute name="NAME" x="309.88" y="109.728" size="1.778" layer="95" font="vector"/>
+</instance>
+<instance part="J2" gate="G$1" x="68.58" y="27.94" smashed="yes">
+<attribute name="VALUE" x="63.5" y="20.574" size="1.778" layer="96" font="vector"/>
+<attribute name="NAME" x="63.5" y="36.068" size="1.778" layer="95" font="vector"/>
 </instance>
 </instances>
@@
 <pinref part="SUPPLY1" gate="GND" pin="GND"/>
 </segment>
+<segment>
+<pinref part="J2" gate="G$1" pin="1"/>
+<wire x1="73.66" y1="25.4" x2="76.2" y2="25.4" width="0.1524" layer="91"/>
+<label x="76.2" y="25.4" size="0.8128" layer="95" xref="yes"/>
+</segment>
+<segment>
+<pinref part="J4" gate="G$1" pin="1"/>
+<wire x1="320.04" y1="99.06" x2="322.58" y2="99.06" width="0.1524" layer="91"/>
+<label x="322.58" y="99.06" size="0.8128" layer="95" xref="yes"/>
+</segment>
+<segment>
+<pinref part="J3" gate="G$1" pin="1"/>
+<wire x1="320.04" y1="124.46" x2="322.58" y2="124.46" width="0.1524" layer="91"/>
+<label x="322.58" y="124.46" size="0.8128" layer="95" xref="yes"/>
+</segment>
+<segment>
+<pinref part="J3" gate="G$1" pin="4"/>
+<wire x1="320.04" y1="132.08" x2="322.58" y2="132.08" width="0.1524" layer="91"/>
+<label x="322.58" y="132.08" size="0.8128" layer="95" xref="yes"/>
+</segment>
+<segment>
+<pinref part="J3" gate="G$1" pin="9"/>
+<wire x1="320.04" y1="144.78" x2="322.58" y2="144.78" width="0.1524" layer="91"/>
+<label x="322.58" y="144.78" size="0.8128" layer="95" xref="yes"/>
+</segment>
 </net>
 <net name="VCC" class="2">
@@
 <wire x1="238.76" y1="157.48" x2="238.76" y2="160.02" width="0.1524" layer="91"/>
 <label x="238.76" y="160.02" size="0.8128" layer="95" rot="R90" xref="yes"/>
+</segment>
+<segment>
+<pinref part="J2" gate="G$1" pin="2"/>
+<wire x1="73.66" y1="27.94" x2="76.2" y2="27.94" width="0.1524" layer="91"/>
+<label x="76.2" y="27.94" size="0.8128" layer="95" xref="yes"/>
 </segment>
 </net>
@@
 <label x="68.58" y="203.2" size="0.8128" layer="95" rot="MR0" xref="yes"/>
 </segment>
+<segment>
+<pinref part="J3" gate="G$1" pin="3"/>
+<wire x1="320.04" y1="129.54" x2="322.58" y2="129.54" width="0.1524" layer="91"/>
+<label x="322.58" y="129.54" size="0.8128" layer="95" xref="yes"/>
+</segment>
 </net>
 <net name="THS" class="0">
@@
 <wire x1="76.2" y1="88.9" x2="73.66" y2="86.36" width="0.1524" layer="91" curve="90"/>
 <wire x1="73.66" y1="86.36" x2="73.66" y2="83.82" width="0.1524" layer="91"/>
+</segment>
+<segment>
+<pinref part="J4" gate="G$1" pin="3"/>
+<wire x1="320.04" y1="104.14" x2="322.58" y2="104.14" width="0.1524" layer="91"/>
+<label x="322.58" y="104.14" size="0.8128" layer="95" xref="yes"/>
 </segment>
 </net>
@@
 <label x="99.06" y="218.44" size="0.8128" layer="95" xref="yes"/>
 </segment>
+<segment>
+<pinref part="J4" gate="G$1" pin="4"/>
+<wire x1="320.04" y1="106.68" x2="322.58" y2="106.68" width="0.1524" layer="91"/>
+<label x="322.58" y="106.68" size="0.8128" layer="95" xref="yes"/>
+</segment>
 </net>
 <net name="DTCT1" class="0">
@@
 <wire x1="96.52" y1="231.14" x2="99.06" y2="231.14" width="0.1524" layer="91"/>
 <label x="99.06" y="231.14" size="0.8128" layer="95" xref="yes"/>
-</segment>
-<segment>
-<pinref part="R5" gate="G$1" pin="2"/>
-<wire x1="279.4" y1="109.22" x2="281.94" y2="109.22" width="0.1524" layer="91"/>
-<label x="281.94" y="109.22" size="0.8128" layer="95" xref="yes"/>
 </segment>
 </net>
@@
 <label x="99.06" y="223.52" size="0.8128" layer="95" xref="yes"/>
 </segment>
+<segment>
+<pinref part="J2" gate="G$1" pin="4"/>
+<wire x1="73.66" y1="33.02" x2="76.2" y2="33.02" width="0.1524" layer="91"/>
+<label x="76.2" y="33.02" size="0.8128" layer="95" xref="yes"/>
+</segment>
 </net>
 <net name="GPIO0" class="0">
@@
 <label x="99.06" y="215.9" size="0.8128" layer="95" xref="yes"/>
 </segment>
+<segment>
+<pinref part="J2" gate="G$1" pin="3"/>
+<wire x1="73.66" y1="30.48" x2="76.2" y2="30.48" width="0.1524" layer="91"/>
+<label x="76.2" y="30.48" size="0.8128" layer="95" xref="yes"/>
+</segment>
 </net>
 <net name="VIN" class="5">
@@
 <label x="236.22" y="63.5" size="0.8128" layer="95" rot="R90" xref="yes"/>
 </segment>
-</net>
-<net name="LED1A" class="0">
-<segment>
-<pinref part="R5" gate="G$1" pin="1"/>
-<wire x1="269.24" y1="109.22" x2="254" y2="109.22" width="0.1524" layer="91"/>
-<label x="261.62" y="109.22" size="1.778" layer="95"/>
+<segment>
+<pinref part="J4" gate="G$1" pin="2"/>
+<wire x1="320.04" y1="101.6" x2="322.58" y2="101.6" width="0.1524" layer="91"/>
+<label x="322.58" y="101.6" size="0.8128" layer="95" xref="yes"/>
 </segment>
 </net>
@@
 <label x="213.36" y="121.92" size="0.8128" layer="95" xref="yes"/>
 <pinref part="RN4" gate="B" pin="2"/>
+</segment>
+<segment>
+<pinref part="J3" gate="G$1" pin="6"/>
+<wire x1="320.04" y1="137.16" x2="322.58" y2="137.16" width="0.1524" layer="91"/>
+<label x="322.58" y="137.16" size="0.8128" layer="95" xref="yes"/>
 </segment>
 </net>
@@
 <pinref part="OK1" gate="A" pin="C1"/>
 </segment>
+<segment>
+<pinref part="J3" gate="G$1" pin="7"/>
+<wire x1="320.04" y1="139.7" x2="322.58" y2="139.7" width="0.1524" layer="91"/>
+<label x="322.58" y="139.7" size="0.8128" layer="95" xref="yes"/>
+</segment>
 </net>
 <net name="MORTN" class="0">
@@
 <pinref part="RN4" gate="F" pin="2"/>
 </segment>
+<segment>
+<pinref part="J3" gate="G$1" pin="10"/>
+<wire x1="320.04" y1="147.32" x2="322.58" y2="147.32" width="0.1524" layer="91"/>
+<label x="322.58" y="147.32" size="0.8128" layer="95" xref="yes"/>
+</segment>
 </net>
 <net name="MOSND" class="0">
@@
 <wire x1="210.82" y1="33.02" x2="205.74" y2="33.02" width="0.1524" layer="91"/>
 <pinref part="RN4" gate="E" pin="2"/>
+</segment>
+<segment>
+<pinref part="J3" gate="G$1" pin="8"/>
+<wire x1="320.04" y1="142.24" x2="322.58" y2="142.24" width="0.1524" layer="91"/>
+<label x="322.58" y="142.24" size="0.8128" layer="95" xref="yes"/>
 </segment>
 </net>
@@
 <wire x1="33.02" y1="190.5" x2="33.02" y2="180.34" width="0.1524" layer="91"/>
 <label x="33.02" y="180.34" size="0.8128" layer="95" rot="R270" xref="yes"/>
+</segment>
+<segment>
+<pinref part="J3" gate="G$1" pin="2"/>
+<wire x1="320.04" y1="127" x2="322.58" y2="127" width="0.1524" layer="91"/>
+<label x="322.58" y="127" size="0.8128" layer="95" xref="yes"/>
 </segment>
 </net>
@@
 </segment>
 </net>
+<net name="LDE0A" class="0">
+<segment>
+<pinref part="J3" gate="G$1" pin="5"/>
+<wire x1="320.04" y1="134.62" x2="322.58" y2="134.62" width="0.1524" layer="91"/>
+<label x="322.58" y="134.62" size="0.8128" layer="95" xref="yes"/>
+</segment>
+</net>
